File: pcb/pompyboard.kicad_sch (KiCad schematic)
At the start: 17 parts, among them J1 USB_C_Receptacle_USB2.0_16P, J2 Conn_01x04_Pin, SW1 EVQQ2B03W, U229 STM32F429IGT6, U230 USB3320C-EZK-TR, U231 AMS1117CD-3.3

Commit message: pcb: use component from jlcpcb "basic" part instead of "extended" (reduce cost from $242.46 to $222.80)
Parts:
- C21, C23, C25: footprint Capacitor_SMD:C_0201_0603Metric -> Capacitor_SMD:C_0402_1005Metric; LCSC Part # C160831 -> C1525
- R1: footprint Resistor_SMD:R_0201_0603Metric -> Resistor_SMD:R_0402_1005Metric; LCSC Part # C473048 -> C25744
- R2, R3: footprint Resistor_SMD:R_0201_0603Metric -> Resistor_SMD:R_0402_1005Metric; LCSC Part # C270344 -> C25905
- R4: footprint Resistor_SMD:R_0201_0603Metric -> Resistor_SMD:R_0402_1005Metric; LCSC Part # C270365 -> C11702
Changed lines of the file:
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@@
 			)
 		)
-		(property "Footprint" "Resistor_SMD:R_0201_0603Metric"
+		(property "Footprint" "Resistor_SMD:R_0402_1005Metric"
 			(at 218.948 59.69 90)
 			(effects
@@
 			)
 		)
-		(property "LCSC Part #" "C270344"
+		(property "LCSC Part #" "C25905"
 			(at 217.17 59.69 0)
 			(effects
@@
 			)
 		)
-		(property "Footprint" "Resistor_SMD:R_0201_0603Metric"
+		(property "Footprint" "Resistor_SMD:R_0402_1005Metric"
 			(at 121.412 218.44 90)
 			(effects
@@
 			)
 		)
-		(property "LCSC Part #" "C473048"
+		(property "LCSC Part #" "C25744"
 			(at 123.19 218.44 0)
 			(effects
@@
 			)
 		)
-		(property "Footprint" "Resistor_SMD:R_0201_0603Metric"
+		(property "Footprint" "Resistor_SMD:R_0402_1005Metric"
 			(at 224.282 64.77 90)
 			(effects
@@
 			)
 		)
-		(property "LCSC Part #" "C270365"
+		(property "LCSC Part #" "C11702"
 			(at 226.06 64.77 0)
 			(effects
@@
 			)
 		)
-		(property "Footprint" "Capacitor_SMD:C_0201_0603Metric"
+		(property "Footprint" "Capacitor_SMD:C_0402_1005Metric"
 			(at 367.9952 43.18 0)
 			(effects
@@
 			)
 		)
-		(property "LCSC Part #" "C160831"
+		(property "LCSC Part #" "C1525"
 			(at 367.03 39.37 0)
 			(effects
@@
 			)
 		)
-		(property "Footprint" "Resistor_SMD:R_0201_0603Metric"
+		(property "Footprint" "Resistor_SMD:R_0402_1005Metric"
 			(at 211.582 74.93 90)
 			(effects
@@
 			)
 		)
-		(property "LCSC Part #" "C270344"
+		(property "LCSC Part #" "C25905"
 			(at 213.36 74.93 0)
 			(effects
@@
 			)
 		)
-		(property "Footprint" "Capacitor_SMD:C_0201_0603Metric"
+		(property "Footprint" "Capacitor_SMD:C_0402_1005Metric"
 			(at 328.6252 43.18 0)
 			(effects
@@
 			)
 		)
-		(property "LCSC Part #" "C160831"
+		(property "LCSC Part #" "C1525"
 			(at 327.66 39.37 0)
 			(effects
@@
 			)
 		)
-		(property "Footprint" "Capacitor_SMD:C_0201_0603Metric"
+		(property "Footprint" "Capacitor_SMD:C_0402_1005Metric"
 			(at 234.6452 44.45 0)
 			(effects
@@
 			)
 		)
-		(property "LCSC Part #" "C160831"
+		(property "LCSC Part #" "C1525"
 			(at 233.68 40.64 0)
 			(effects

Commit message: pcb: fix LED footprint not matching actual component
Parts:
- D1: footprint LED_SMD:LED_0201_0603Metric -> LED_SMD:LED_0603_1608Metric
Changed lines of the file:
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@@
 			)
 		)
-		(property "Footprint" "LED_SMD:LED_0201_0603Metric"
+		(property "Footprint" "LED_SMD:LED_0603_1608Metric"
 			(at 226.06 72.39 0)
 			(effects

Commit message: pcb: pull down BOOT0 to make the board programmable via ST-Link
Connections:
- net GND: now also U229.166 (BOOT0)
- no-connect marks 125 -> 124
Changed lines of the file:
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@@
 	)
 	(no_connect
-		(at 27.94 54.61)
-	)
-	(no_connect
 		(at 27.94 214.63)
 	)
@@
 		)
 	)
+	(wire
+		(pts
+			(xy 24.13 54.61) (xy 27.94 54.61)
+		)
+		(stroke
+			(width 0)
+			(type default)
+		)
+	)
 	(polyline
 		(pts
@@
 					(unit 1)
 				)
+			)
+		)
+	)
+	(symbol
+		(lib_id "power:GND")
+		(at 24.13 54.61 0)
+		(unit 1)
+		(exclude_from_sim no)
+		(in_bom yes)
+		(on_board yes)
+		(dnp no)
+		(fields_autoplaced yes)
+		(property "Reference" "#PWR06"
+			(at 24.13 60.96 0)
+			(effects
+				(font
+					(size 1.27 1.27)
+				)
+				(hide yes)
+			)
+		)
+		(property "Value" "GND"
+			(at 24.13 59.69 0)
+			(effects
+				(font
+					(size 1.27 1.27)
+				)
+			)
+		)
+		(property "Footprint" ""
+			(at 24.13 54.61 0)
+			(effects
+				(font
+					(size 1.27 1.27)
+				)
+				(hide yes)
+			)
+		)
+		(property "Datasheet" ""
+			(at 24.13 54.61 0)
+			(effects
+				(font
+					(size 1.27 1.27)
+				)
+				(hide yes)
+			)
+		)
+		(property "Description" "Power symbol creates a global label with name \"GND\" , ground"
+			(at 24.13 54.61 0)
+			(effects
+				(font
+					(size 1.27 1.27)
+				)
+				(hide yes)
+			)
+		)
+		(pin "1"
+		)
+		(instances
+			(project "pompyboard"
+				(path "/e5830f2e-b6bc-440e-bdf9-7651ab21e3a0"
+					(reference "#PWR06")
+					(unit 1)
+				)

Commit message: pcb: connect vref to 3.3v
Connections:
- net 3.3V: now also U229.38 (VREF+)
- no-connect marks 124 -> 123
Changed lines of the file:
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@@
 	)
 	(no_connect
-		(at 27.94 59.69)
-	)
-	(no_connect
 		(at 27.94 229.87)
 	)
@@
 		)
 	)
-	(wire
-		(pts
-			(xy 24.13 54.61) (xy 27.94 54.61)
-		)
-		(stroke
-			(width 0)
-			(type default)
-		)
-	)
 	(polyline
 		(pts
@@
 		)
 	)
+	(wire
+		(pts
+			(xy 17.78 54.61) (xy 27.94 54.61)
+		)
+		(stroke
+			(width 0)
+			(type default)
+		)
+	)
 	(polyline
 		(pts
@@
 		)
 	)
+	(global_label "3.3V"
+		(shape input)
+		(at 27.94 59.69 180)
+		(fields_autoplaced yes)
+		(effects
+			(font
+				(size 1.27 1.27)
+			)
+			(justify right)
+		)
+		(property "Intersheetrefs" "${INTERSHEET_REFS}"
+			(at 20.8424 59.69 0)
+			(effects
+				(font
+					(size 1.27 1.27)
+				)
+				(justify right)
+				(hide yes)
+			)
+		)
+	)
 	(global_label "MUX14_OUT"
 		(shape input)
@@
 	(symbol
 		(lib_id "power:GND")
-		(at 24.13 54.61 0)
+		(at 17.78 54.61 0)
 		(unit 1)
 		(exclude_from_sim no)
@@
 		(fields_autoplaced yes)
 		(property "Reference" "#PWR06"
-			(at 24.13 60.96 0)
+			(at 17.78 60.96 0)
 			(effects
 				(font
@@
 		)
 		(property "Value" "GND"
-			(at 24.13 59.69 0)
+			(at 17.78 59.69 0)
 			(effects
 				(font
@@
 		)
 		(property "Footprint" ""
-			(at 24.13 54.61 0)
+			(at 17.78 54.61 0)
 			(effects
 				(font
@@
 		)
 		(property "Datasheet" ""
-			(at 24.13 54.61 0)
+			(at 17.78 54.61 0)
 			(effects
 				(font
@@
 		)
 		(property "Description" "Power symbol creates a global label with name \"GND\" , ground"
-			(at 24.13 54.61 0)
+			(at 17.78 54.61 0)
 			(effects
 				(font

Commit message: pcb: remove usb controller (work with 1000Hz polling rate for now)
Parts:
- removed C20: 10u, Capacitor_SMD:C_0603_1608Metric, symbol Device:C
- removed C21: 0.1u, Capacitor_SMD:C_0402_1005Metric, symbol Device:C
- removed U230: USB3320C-EZK-TR, Package_DFN_QFN:QFN-32-1EP_5x5mm_P0.5mm_EP3.45x3.45mm, symbol Interface_USB:USB3300-EZK
Connections:
- net D+: now also U229.123 (PA12)
- net D-: now also U229.122 (PA11)
- net MCO: no longer names the net of U229.118 (PC9)
- net ULPI_CK: no longer names the net of U229.51 (PA5)
- net ULPI_D0: no longer names the net of U229.44 (PH3)
- net ULPI_D1: no longer names the net of U229.56 (PB0)
- net ULPI_D2: no longer names the net of U229.57 (PB1)
- net ULPI_D3: no longer names the net of U229.79 (PB10)
- net ULPI_D4: no longer names the net of U229.80 (PB11)
- net ULPI_D5: no longer names the net of U229.92 (PB12)
- net ULPI_D6: no longer names the net of U229.93 (PB13)
- net ULPI_D7: no longer names the net of U229.163 (PB5)
- net ULPI_DIR: no longer names the net of U229.13 (PI11)
- net ULPI_NXT: no longer names the net of U229.45 (PH4)
- net ULPI_STP: no longer names the net of U229.32 (PC0)
- no-connect marks 123 -> 120
Other:
- note added: "ADC123_IN10"
- note added: "ADC123_IN12"
- note added: "ADC123_IN13"
- note added: "ADC12_IN5"
- note added: "ADC12_IN8"
- note added: "ADC12_IN9"
- note added: "OTG_FS_DM"
- note added: "OTG_FS_DP"
- note removed: "MCO2"
- note removed: "OSC_IN"
- note removed: "OTG_HS_ULPI_CK/ADC12_IN5"
- note removed: "OTG_HS_ULPI_D0"
- note removed: "OTG_HS_ULPI_D1/ADC12_IN8"
- note removed: "OTG_HS_ULPI_D2/ADC12_IN9"
- note removed: "OTG_HS_ULPI_D3"
- note removed: "OTG_HS_ULPI_D4"
- note removed: "OTG_HS_ULPI_D5"
- note removed: "OTG_HS_ULPI_D6"
- note removed: "OTG_HS_ULPI_D7"
- note removed: "OTG_HS_ULPI_DIR"
- note removed: "OTG_HS_ULPI_DIR/ADC123_IN12"
- note removed: "OTG_HS_ULPI_NXT"
- note removed: "OTG_HS_ULPI_NXT/ADC123_IN13"
- note removed: "OTG_HS_ULPI_STP/ADC123_IN10"
- moved on the sheet: C22, C23, C24, C25, D1, R4, U231
